Commit message: cannot work

File: workspace/arm_ws2/src/small_arm_description/urdf/small_arm.urdf (robot description, URDF)
Before this commit: robot small_arm, 11 links, 10 joints
Links:
- removed link base_link
- added link base_arm, mass 1.29137439344346; collision mesh filename=/home/taiting/docker_ws/timda_dual_arm_ws/src/tb4_arm_ros2/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 scale=0.001 0.001 0.001; visual mesh filename=/home/taiting/docker_ws/timda_dual_arm_ws/src/tb4_arm_ros2/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 scale=0.001 0.001 0.001
Joints:
- removed joint origin_to_base_link
- added joint origin_to_base_arm: type fixed, parent world, child base_arm, origin xyz=0 0 0 rpy=0 0 0, axis 0 0 0
- joint joint1: parent base_link -> base_arm

File: workspace/arm_ws2/src/small_arm_description/urdf/small_arm.xacro (robot description, xacro)
@@ -4,6 +4,6 @@
   <!-- <xacro:include filename="$(find SMW-G02_urdf_description)/urdf/SMW-G02_urdf.trans" />
   <xacro:include filename="$(find SMW-G02_urdf_description)/urdf/SMW-G02_urdf.gazebo" /> -->
-  <xacro:macro name="small_arm" params="parent base_name:=base_link *origin">
-  <joint name="origin_to_base_link" type="fixed">
+  <xacro:macro name="small_arm" params="parent base_name:=base_arm *origin">
+  <joint name="origin_to_base_arm" type="fixed">
     <xacro:insert_block name="origin" />
     <parent link="${parent}" />

File: workspace/arm_ws2/src/small_arm_moveit_config/config/small_arm.ros2_control.xacro (robot description, xacro)
@@ -10,5 +10,5 @@
                 <xacro:if value="${ros2_control_hardware_type == 'real'}">
                     <plugin>dynamixel_hardware/DynamixelHardware</plugin>
-                    <param name="usb_port">/dev/ttyUSB0</param>
+                    <param name="usb_port">/dev/serial/by-id/usb-FTDI_USB__-__Serial_Converter_FT88Z12T-if00-port0</param>
                     <param name="baud_rate">115200</param>
                     <param name="use_dummy">false</param>
